Commit message: Add frames for imu and velodyne
Signed-off-by: Shrijit Singh <shrijitsingh99@gmail.com>

File: launchers/urdf/test_rig.urdf (robot description, URDF)
Before this commit: robot test_rig, 5 links, 4 joints
Links:
- removed link lidar_link
- added link velodyne; visual cylinder length=0.071 radius=0.0515
- added link xsens_imu
Joints:
- removed joint imu_lidar_joint
- added joint imu_velodyne_joint: type fixed, parent imu_link, child velodyne, origin xyz=0 0 -0.081445 rpy=0 3.14 -3.14
- joint base_link_imu_joint: child imu_link -> xsens_imu; origin xyz=0 0 0 rpy=0 2.8797 -3.14 -> xyz=0 0 0 rpy=0 0 0; parent base_link -> imu_link

Commit message: Fix joint name duplication issue
Signed-off-by: Shrijit Singh <shrijitsingh99@gmail.com>

File: launchers/urdf/test_rig.urdf (robot description, URDF)
Before this commit: robot test_rig, 6 links, 4 joints
Joints:
- added joint imu_xsens_imu_joint: type fixed, parent imu_link, child xsens_imu, origin xyz=0 0 0 rpy=0 0 0
- joint base_link_imu_joint: child xsens_imu -> imu_link; origin xyz=0 0 0 rpy=0 0 0 -> xyz=0 0 0 rpy=0 2.8797 -3.14; parent imu_link -> base_link

Commit message: Add gps link
Signed-off-by: Shrijit Singh <shrijitsingh99@gmail.com>

File: launchers/urdf/test_rig.urdf (robot description, URDF)
Before this commit: robot test_rig, 6 links, 5 joints
Links:
- added link gps; visual box size=0.0364 .0364 0.02325
Joints:
- added joint base_link_gps_joint: type fixed, parent base_link, child gps, origin xyz=-0.4 0 -0.05 rpy=0 0 0
